File: kicad/b2b_converter.kicad_pcb (KiCad board)
At the start: 4 copper layers, 340 x 240 mm, 233 parts, among them J1 RED 3~ + PE, J10 HALL AIN_IAFE_A, J11 HALL AIN_IAFE_B, J12 HALL AIN_IAFE_C, J13 HALL AIN_IMOT_U, J14 HALL AIN_IMOT_V, J15 HALL AIN_IMOT_W, J20 SWD, J3 R FRENADO, J30 CONTACTOR LINEA K1, J31 BYPASS PRECARGA K2, J32 VENTILADOR, J33 E-STOP, J4 MOTOR U/V/W/PE, J40 24 Vdc IN, J50 DCDC ISO 15V rama 1, J51 DCDC ISO 15V rama 2, J52 DCDC ISO 15V rama 3, J53 DCDC ISO 15V rama 4, J54 DCDC ISO 15V rama 5, J55 DCDC ISO 15V rama 6, J60 CAMPO / ETHERNET, K2 BYPASS PRECARGA, Q1 C3M0075120K, Q10 C3M0075120K, Q11 C3M0075120K, Q12 C3M0075120K, Q2 C3M0075120K, Q20 AO3400, Q21 AO3400, Q22 AO3400, Q3 C3M0075120K, Q4 C3M0075120K, Q5 C3M0075120K, Q6 C3M0075120K, Q7 C3M0075120K, Q8 C3M0075120K, Q9 C3M0075120K, SW1 NRST, SW60 ESP_EN, SW61 ESP_BOOT, U1 STM32G474VET6, U11 UCC21520DW, U12 UCC21520DW, U13 UCC21520DW, U14 UCC21520DW, U15 UCC21520DW, U16 UCC21520DW, U20 LM358, U30 LM339, U40 LMR33630 24->15V, U41 LMR33630 15->5V, U42 TLV75833 5->3V3, U50 ADuM1401ARWZ, U60 ESP32-S3-WROOM-1-N8, X1 24MHz

Commit message: Corrige tres bugs de conectividad del bus DC y anade guia de simulacion
Al intentar rutear los lazos de conmutacion aparecieron tres errores graves
del esquematico que ninguna revision visual habia detectado:

1. Los rieles del bus DC solo conectaban la ULTIMA rama de cada puente.
   DC_P tenia 4 pads en vez de 22; Q1, Q3, Q7 y Q9 quedaban unconnected.
   Causa: el riel era un unico cable largo y los stubs de cada rama morian
   en mitad de el. KiCad solo une cables extremo con extremo: un cable que
   termina en medio de otro NO conecta, ni con junction. Solo funcionaba la
   ultima rama porque coincidia con el extremo del riel.
   Corregido con un helper rail() que construye el riel PARTIDO en cada
   punto de contacto.

2. El puente AFE no estaba conectado al filtro LCL: el nodo de conmutacion
   se llamaba SW_A y la salida del LCL AFE_A. Mismo nodo fisico, dos
   nombres. Unificado a AFE_A/B/C.

3. La resistencia de precarga quedaba puenteada porque el helper de riel
   se tragaba tambien el nodo DC_RAW. Corregido acotando con xmin.

Resultado: DC_P de 4 a 22 pads, DC_N de 4 a 18.

Tambien: se probo extender el bus laminado sobre toda la fila de potencia y
EMPEORA (293 clearance, 34 cortos): con 3 mm exigidos a HV_DC y los pines
del TO-247-4 a 2.54 mm el plano no cabe entre drenador y puerta. Revertido y
documentado.

Nuevo: docs/COMO_SIMULAR.md con las cuatro simulaciones del proyecto.

Co-Authored-By: Claude Opus 5 <noreply@anthropic.com>
Connections:
- C1 pad 1: (no net) -> DC_P
- C2 pad 1: (no net) -> DC_P
- C2 pad 2: (no net) -> DC_N
- C3 pad 1: (no net) -> DC_P
- C3 pad 2: (no net) -> DC_N
- C4 pad 1: (no net) -> DC_P
- C4 pad 2: (no net) -> DC_N
- CDA pad 1: (no net) -> DC_P
- CDA pad 2: (no net) -> DC_N
- CDB pad 1: (no net) -> DC_P
- CDB pad 2: (no net) -> DC_N
- CDC pad 1: (no net) -> DC_P
- CDC pad 2: (no net) -> DC_N
- CDU pad 1: (no net) -> DC_P
- CDU pad 2: (no net) -> DC_N
- CDV pad 1: (no net) -> DC_P
- CDV pad 2: (no net) -> DC_N
- CDW pad 1: (no net) -> DC_P
- CDW pad 2: (no net) -> DC_N
- CFA pad 1: (no net) -> Net-(CFA-Pad1)
- CFB pad 1: (no net) -> Net-(CFB-Pad1)
- CFC pad 1: (no net) -> Net-(CFC-Pad1)
- D1 pad 1: (no net) -> Net-(D1-K)
- D1 pad 2: (no net) -> DC_N
- D20 pad 2: (no net) -> Net-(D20-A)
- D21 pad 2: (no net) -> Net-(D21-A)
- D22 pad 2: (no net) -> Net-(D22-A)
- D30 pad 1: (no net) -> Net-(D30-K)
- D31 pad 1: (no net) -> Net-(D31-K)
- D60 pad 1: (no net) -> Net-(D60-K)
- D61 pad 1: (no net) -> Net-(D61-K)
- DBRK pad 1: (no net) -> DC_P
- DBRK pad 2: (no net) -> Net-(DBRK-A)
- DGH1 pad 2: (no net) -> Net-(DGH1-A)
- DGH2 pad 2: (no net) -> Net-(DGH2-A)
- DGH3 pad 2: (no net) -> Net-(DGH3-A)
- DGH4 pad 2: (no net) -> Net-(DGH4-A)
- DGH5 pad 2: (no net) -> Net-(DGH5-A)
- DGH6 pad 2: (no net) -> Net-(DGH6-A)
- DGL1 pad 2: (no net) -> Net-(DGL1-A)
- DGL2 pad 2: (no net) -> Net-(DGL2-A)
- DGL3 pad 2: (no net) -> Net-(DGL3-A)
- DGL4 pad 2: (no net) -> Net-(DGL4-A)
- DGL5 pad 2: (no net) -> Net-(DGL5-A)
- DGL6 pad 2: (no net) -> Net-(DGL6-A)
- F1 pad 1: (no net) -> Net-(J1-Pin_1)
- F1 pad 2: (no net) -> Net-(F1-Pad2)
- F2 pad 1: (no net) -> Net-(J1-Pin_2)
- F2 pad 2: (no net) -> Net-(F2-Pad2)
- F3 pad 1: (no net) -> Net-(J1-Pin_3)
- F3 pad 2: (no net) -> Net-(F3-Pad2)
- J1 pad 1: (no net) -> Net-(J1-Pin_1)
- J1 pad 2: (no net) -> Net-(J1-Pin_2)
- J1 pad 3: (no net) -> Net-(J1-Pin_3)
- J10 pad 2: (no net) -> Net-(J10-Pin_2)
- J11 pad 2: (no net) -> Net-(J11-Pin_2)
- J12 pad 2: (no net) -> Net-(J12-Pin_2)
- J13 pad 2: (no net) -> Net-(J13-Pin_2)
- J14 pad 2: (no net) -> Net-(J14-Pin_2)
- J15 pad 2: (no net) -> Net-(J15-Pin_2)
- J3 pad 1: (no net) -> Net-(DBRK-A)
- J30 pad 2: (no net) -> Net-(D20-A)
- J31 pad 2: (no net) -> Net-(D21-A)
- J32 pad 2: (no net) -> Net-(D22-A)
- L1A pad 1: (no net) -> Net-(L1A-Pad1)
- L1B pad 1: (no net) -> Net-(L1B-Pad1)
- L1C pad 1: (no net) -> Net-(L1C-Pad1)
- L2A pad 1: (no net) -> Net-(L2A-Pad1)
- L2A pad 2: (no net) -> Net-(L1A-Pad1)
- L2B pad 1: (no net) -> Net-(L2B-Pad1)
- L2B pad 2: (no net) -> Net-(L1B-Pad1)
- L2C pad 1: (no net) -> Net-(L2C-Pad1)
- L2C pad 2: (no net) -> Net-(L1C-Pad1)
- LCM1 pad 1: (no net) -> Net-(F1-Pad2)
- LCM1 pad 2: (no net) -> Net-(L2A-Pad1)
- LCM2 pad 1: (no net) -> Net-(F2-Pad2)
- LCM2 pad 2: (no net) -> Net-(L2B-Pad1)
- LCM3 pad 1: (no net) -> Net-(F3-Pad2)
- LCM3 pad 2: (no net) -> Net-(L2C-Pad1)
- Q1 pad 1: (no net) -> DC_P
- Q1 pad 2: SW_A -> AFE_A
- Q10 pad 2: (no net) -> DC_N
- Q2 pad 1: SW_A -> AFE_A
- Q2 pad 2: (no net) -> DC_N
- Q20 pad 2: (no net) -> Net-(D20-A)
- Q21 pad 2: (no net) -> Net-(D21-A)
- Q22 pad 2: (no net) -> Net-(D22-A)
- Q3 pad 1: (no net) -> DC_P
- Q3 pad 2: SW_B -> AFE_B
- Q4 pad 1: SW_B -> AFE_B
- Q4 pad 2: (no net) -> DC_N
- Q5 pad 2: SW_C -> AFE_C
- Q6 pad 1: SW_C -> AFE_C
- Q7 pad 1: (no net) -> DC_P
- Q8 pad 2: (no net) -> DC_N
- Q9 pad 1: (no net) -> DC_P
- QBRK pad 1: (no net) -> DC_P
- QBRK pad 2: (no net) -> Net-(DBRK-A)
- RB1 pad 1: (no net) -> Net-(J10-Pin_2)
- RB1A pad 1: (no net) -> Net-(J10-Pin_2)
- RB1A pad 2: (no net) -> Net-(RB1A-Pad2)
- RB1B pad 1: (no net) -> Net-(RB1A-Pad2)
- RB1C pad 1: (no net) -> Net-(RB1A-Pad2)
- RB2 pad 1: (no net) -> Net-(J11-Pin_2)
- RB2A pad 1: (no net) -> Net-(J11-Pin_2)
- RB2A pad 2: (no net) -> Net-(RB2A-Pad2)
- RB2B pad 1: (no net) -> Net-(RB2A-Pad2)
- RB2C pad 1: (no net) -> Net-(RB2A-Pad2)
- RB3 pad 1: (no net) -> Net-(J12-Pin_2)
- RB3A pad 1: (no net) -> Net-(J12-Pin_2)
- RB3A pad 2: (no net) -> Net-(RB3A-Pad2)
- RB3B pad 1: (no net) -> Net-(RB3A-Pad2)
- RB3C pad 1: (no net) -> Net-(RB3A-Pad2)
- RB4 pad 1: (no net) -> Net-(J13-Pin_2)
- RB4A pad 1: (no net) -> Net-(J13-Pin_2)
- RB4A pad 2: (no net) -> Net-(RB4A-Pad2)
- RB4B pad 1: (no net) -> Net-(RB4A-Pad2)
- RB4C pad 1: (no net) -> Net-(RB4A-Pad2)
- RB5 pad 1: (no net) -> Net-(J14-Pin_2)
- RB5A pad 1: (no net) -> Net-(J14-Pin_2)
- RB5A pad 2: (no net) -> Net-(RB5A-Pad2)
- RB5B pad 1: (no net) -> Net-(RB5A-Pad2)
- RB5C pad 1: (no net) -> Net-(RB5A-Pad2)
- RB6 pad 1: (no net) -> Net-(J15-Pin_2)
- RB6A pad 1: (no net) -> Net-(J15-Pin_2)
- RB6A pad 2: (no net) -> Net-(RB6A-Pad2)
- RB6B pad 1: (no net) -> Net-(RB6A-Pad2)
- RB6C pad 1: (no net) -> Net-(RB6A-Pad2)
- RBLEED pad 1: (no net) -> DC_P
- RBLEED pad 2: (no net) -> Net-(RBLEED-Pad2)
- RDA pad 2: (no net) -> Net-(CFA-Pad1)
- RDB pad 2: (no net) -> Net-(CFB-Pad1)
- RDC pad 2: (no net) -> Net-(CFC-Pad1)
- RDT1 pad 1: (no net) -> Net-(U11-DT)
- RDT2 pad 1: (no net) -> Net-(U12-DT)
- RDT3 pad 1: (no net) -> Net-(U13-DT)
- RDT4 pad 1: (no net) -> Net-(U14-DT)
- RDT5 pad 1: (no net) -> Net-(U15-DT)
- RDT6 pad 1: (no net) -> Net-(U16-DT)
- RDV1 pad 1: (no net) -> DC_P
- RDV1 pad 2: (no net) -> Net-(RDV1-Pad2)
- RDV2 pad 1: (no net) -> Net-(RDV1-Pad2)
- RDV2 pad 2: (no net) -> Net-(RDV2-Pad2)
- RDV3 pad 1: (no net) -> Net-(RDV2-Pad2)
- RDV3 pad 2: (no net) -> Net-(RDV3-Pad2)
- RDV4 pad 1: (no net) -> Net-(RDV3-Pad2)
- RDV4 pad 2: (no net) -> Net-(RDV4-Pad2)
- RDV5 pad 1: (no net) -> Net-(RDV4-Pad2)
- RDV6 pad 1: (no net) -> unconnected-(RDV6-Pad1)
- RDV6 pad 2: (no net) -> unconnected-(RDV6-Pad2)
- RGH1 pad 1: (no net) -> Net-(U11-OUTA)
- RGH2 pad 1: (no net) -> Net-(U12-OUTA)
- RGH3 pad 1: (no net) -> Net-(U13-OUTA)
- RGH4 pad 1: (no net) -> Net-(U14-OUTA)
- RGH5 pad 1: (no net) -> Net-(U15-OUTA)
- RGH6 pad 1: (no net) -> Net-(U16-OUTA)
- RGL1 pad 1: (no net) -> Net-(U11-OUTB)
- RGL2 pad 1: (no net) -> Net-(U12-OUTB)
- RGL3 pad 1: (no net) -> Net-(U13-OUTB)
- RGL4 pad 1: (no net) -> Net-(U14-OUTB)
- RGL5 pad 1: (no net) -> Net-(U15-OUTB)
- RGL6 pad 1: (no net) -> Net-(U16-OUTB)
- RGOH1 pad 1: (no net) -> Net-(U11-OUTA)
- RGOH1 pad 2: (no net) -> Net-(DGH1-A)
- RGOH2 pad 1: (no net) -> Net-(U12-OUTA)
- RGOH2 pad 2: (no net) -> Net-(DGH2-A)
- RGOH3 pad 1: (no net) -> Net-(U13-OUTA)
- RGOH3 pad 2: (no net) -> Net-(DGH3-A)
- RGOH4 pad 1: (no net) -> Net-(U14-OUTA)
- RGOH4 pad 2: (no net) -> Net-(DGH4-A)
- RGOH5 pad 1: (no net) -> Net-(U15-OUTA)
- RGOH5 pad 2: (no net) -> Net-(DGH5-A)
- RGOH6 pad 1: (no net) -> Net-(U16-OUTA)
- RGOH6 pad 2: (no net) -> Net-(DGH6-A)
- RGOL1 pad 1: (no net) -> Net-(U11-OUTB)
- RGOL1 pad 2: (no net) -> Net-(DGL1-A)
- RGOL2 pad 1: (no net) -> Net-(U12-OUTB)
- RGOL2 pad 2: (no net) -> Net-(DGL2-A)
- RGOL3 pad 1: (no net) -> Net-(U13-OUTB)
- RGOL3 pad 2: (no net) -> Net-(DGL3-A)
- RGOL4 pad 1: (no net) -> Net-(U14-OUTB)
- RGOL4 pad 2: (no net) -> Net-(DGL4-A)
- RGOL5 pad 1: (no net) -> Net-(U15-OUTB)
- RGOL5 pad 2: (no net) -> Net-(DGL5-A)
- RGOL6 pad 1: (no net) -> Net-(U16-OUTB)
- RGOL6 pad 2: (no net) -> Net-(DGL6-A)
- RL0 pad 2: (no net) -> Net-(D30-K)
- RL1 pad 2: (no net) -> Net-(D31-K)
- RL60 pad 2: (no net) -> Net-(D60-K)
- RL61 pad 2: (no net) -> Net-(D61-K)
- RLED pad 1: (no net) -> Net-(RBLEED-Pad2)
- RLED pad 2: (no net) -> Net-(D1-K)
- U1 pad 1: (no net) -> unconnected-(U1-PE2-Pad1)
- U1 pad 10: (no net) -> unconnected-(U1-PF9-Pad10)
- U1 pad 11: (no net) -> unconnected-(U1-PF10-Pad11)
- U1 pad 12: (no net) -> unconnected-(U1-PF0-Pad12)
- U1 pad 13: (no net) -> unconnected-(U1-PF1-Pad13)
- U1 pad 14: (no net) -> unconnected-(U1-PG10-Pad14)
- U1 pad 19: (no net) -> unconnected-(U1-PF2-Pad19)
- U1 pad 2: (no net) -> unconnected-(U1-PE3-Pad2)
- U1 pad 3: (no net) -> unconnected-(U1-PE4-Pad3)
- U1 pad 30: (no net) -> unconnected-(U1-PC4-Pad30)
- U1 pad 31: (no net) -> unconnected-(U1-PC5-Pad31)
- U1 pad 34: (no net) -> unconnected-(U1-PB2-Pad34)
- U1 pad 38: (no net) -> unconnected-(U1-PE7-Pad38)
- U1 pad 4: (no net) -> unconnected-(U1-PE5-Pad4)
- U1 pad 45: (no net) -> unconnected-(U1-PE14-Pad45)
- U1 pad 47: (no net) -> unconnected-(U1-PB10-Pad47)
- U1 pad 5: (no net) -> unconnected-(U1-PE6-Pad5)
- U1 pad 50: (no net) -> unconnected-(U1-PB11-Pad50)
- U1 pad 53: (no net) -> unconnected-(U1-PB14-Pad53)
- U1 pad 54: (no net) -> unconnected-(U1-PB15-Pad54)
- U1 pad 68: (no net) -> unconnected-(U1-PC9-Pad68)
- U1 pad 69: (no net) -> unconnected-(U1-PA8-Pad69)
- U1 pad 7: (no net) -> unconnected-(U1-PC13-Pad7)
- U1 pad 70: (no net) -> unconnected-(U1-PA9-Pad70)
- U1 pad 71: (no net) -> unconnected-(U1-PA10-Pad71)
- U1 pad 72: (no net) -> unconnected-(U1-PA11-Pad72)
- U1 pad 73: (no net) -> unconnected-(U1-PA12-Pad73)
- U1 pad 76: (no net) -> unconnected-(U1-PA13-Pad76)
- U1 pad 77: (no net) -> unconnected-(U1-PA14-Pad77)
- U1 pad 78: (no net) -> unconnected-(U1-PA15-Pad78)
- U1 pad 79: (no net) -> unconnected-(U1-PC10-Pad79)
- U1 pad 8: (no net) -> unconnected-(U1-PC14-Pad8)
- U1 pad 80: (no net) -> unconnected-(U1-PC11-Pad80)
- U1 pad 81: (no net) -> unconnected-(U1-PC12-Pad81)
- U1 pad 82: (no net) -> unconnected-(U1-PD0-Pad82)
- U1 pad 83: (no net) -> unconnected-(U1-PD1-Pad83)
- U1 pad 84: (no net) -> unconnected-(U1-PD2-Pad84)
- U1 pad 89: (no net) -> unconnected-(U1-PD7-Pad89)
- U1 pad 9: (no net) -> unconnected-(U1-PC15-Pad9)
- U1 pad 90: (no net) -> unconnected-(U1-PB3-Pad90)
- U1 pad 94: (no net) -> unconnected-(U1-PB7-Pad94)
- U1 pad 95: (no net) -> unconnected-(U1-PB8-Pad95)
- U1 pad 96: (no net) -> unconnected-(U1-PB9-Pad96)
- U1 pad 97: (no net) -> unconnected-(U1-PE0-Pad97)
- U1 pad 98: (no net) -> unconnected-(U1-PE1-Pad98)
- U11 pad 10: (no net) -> Net-(U11-OUTB)
- U11 pad 12: (no net) -> unconnected-(U11-NC-Pad12)
- U11 pad 13: (no net) -> unconnected-(U11-NC-Pad13)
- U11 pad 15: (no net) -> Net-(U11-OUTA)
- U11 pad 6: (no net) -> Net-(U11-DT)
- U11 pad 7: (no net) -> unconnected-(U11-NC-Pad7)
- U12 pad 10: (no net) -> Net-(U12-OUTB)
- U12 pad 12: (no net) -> unconnected-(U12-NC-Pad12)
- U12 pad 13: (no net) -> unconnected-(U12-NC-Pad13)
- U12 pad 15: (no net) -> Net-(U12-OUTA)
- U12 pad 6: (no net) -> Net-(U12-DT)
- U12 pad 7: (no net) -> unconnected-(U12-NC-Pad7)
- U13 pad 10: (no net) -> Net-(U13-OUTB)
- U13 pad 12: (no net) -> unconnected-(U13-NC-Pad12)
- U13 pad 13: (no net) -> unconnected-(U13-NC-Pad13)
- U13 pad 15: (no net) -> Net-(U13-OUTA)
- U13 pad 6: (no net) -> Net-(U13-DT)
- U13 pad 7: (no net) -> unconnected-(U13-NC-Pad7)
- U14 pad 10: (no net) -> Net-(U14-OUTB)
- U14 pad 12: (no net) -> unconnected-(U14-NC-Pad12)
- U14 pad 13: (no net) -> unconnected-(U14-NC-Pad13)
- U14 pad 15: (no net) -> Net-(U14-OUTA)
- U14 pad 6: (no net) -> Net-(U14-DT)
- U14 pad 7: (no net) -> unconnected-(U14-NC-Pad7)
- U15 pad 10: (no net) -> Net-(U15-OUTB)
- U15 pad 12: (no net) -> unconnected-(U15-NC-Pad12)
- U15 pad 13: (no net) -> unconnected-(U15-NC-Pad13)
- U15 pad 15: (no net) -> Net-(U15-OUTA)
- U15 pad 6: (no net) -> Net-(U15-DT)
- U15 pad 7: (no net) -> unconnected-(U15-NC-Pad7)
- U16 pad 10: (no net) -> Net-(U16-OUTB)
- U16 pad 12: (no net) -> unconnected-(U16-NC-Pad12)
- U16 pad 13: (no net) -> unconnected-(U16-NC-Pad13)
- U16 pad 15: (no net) -> Net-(U16-OUTA)
- U16 pad 6: (no net) -> Net-(U16-DT)
- U16 pad 7: (no net) -> unconnected-(U16-NC-Pad7)
- U20 pad 5: (no net) -> Net-(U20B-+)
- U20 pad 6: (no net) -> Net-(U20B-+)
- U40 pad 4: (no net) -> unconnected-(U40-FB-Pad4)
- U41 pad 4: (no net) -> unconnected-(U41-FB-Pad4)
- U42 pad 4: (no net) -> unconnected-(U42-FB-Pad4)
- U60 pad 13: (no net) -> unconnected-(U60-USB_D--Pad13)
- U60 pad 14: (no net) -> unconnected-(U60-USB_D+-Pad14)
- U60 pad 15: (no net) -> unconnected-(U60-IO3-Pad15)
- U60 pad 16: (no net) -> unconnected-(U60-IO46-Pad16)
- U60 pad 20: (no net) -> unconnected-(U60-IO12-Pad20)
- U60 pad 21: (no net) -> unconnected-(U60-IO13-Pad21)
- U60 pad 22: (no net) -> unconnected-(U60-IO14-Pad22)
- U60 pad 23: (no net) -> unconnected-(U60-IO21-Pad23)
- U60 pad 24: (no net) -> unconnected-(U60-IO47-Pad24)
- U60 pad 25: (no net) -> unconnected-(U60-IO48-Pad25)
- U60 pad 26: (no net) -> unconnected-(U60-IO45-Pad26)
- U60 pad 27: (no net) -> unconnected-(U60-IO0-Pad27)
- U60 pad 28: (no net) -> unconnected-(U60-IO35-Pad28)
- U60 pad 29: (no net) -> unconnected-(U60-IO36-Pad29)
- U60 pad 30: (no net) -> unconnected-(U60-IO37-Pad30)
- U60 pad 31: (no net) -> unconnected-(U60-IO38-Pad31)
- U60 pad 32: (no net) -> unconnected-(U60-IO39-Pad32)
- U60 pad 33: (no net) -> unconnected-(U60-IO40-Pad33)
- U60 pad 34: (no net) -> unconnected-(U60-IO41-Pad34)
- U60 pad 35: (no net) -> unconnected-(U60-IO42-Pad35)
- U60 pad 36: (no net) -> unconnected-(U60-RXD0-Pad36)
- U60 pad 37: (no net) -> unconnected-(U60-TXD0-Pad37)
- U60 pad 38: (no net) -> unconnected-(U60-IO2-Pad38)
- U60 pad 39: (no net) -> unconnected-(U60-IO1-Pad39)
- U60 pad 4: (no net) -> unconnected-(U60-IO4-Pad4)
- U60 pad 5: (no net) -> unconnected-(U60-IO5-Pad5)
- U60 pad 6: (no net) -> unconnected-(U60-IO6-Pad6)
- U60 pad 7: (no net) -> unconnected-(U60-IO7-Pad7)
- U60 pad 8: (no net) -> unconnected-(U60-IO15-Pad8)
- U60 pad 9: (no net) -> unconnected-(U60-IO16-Pad9)

Commit message: Anade protecciones electricas y stackup con color
PROTECCIONES (de 15 a 56 componentes de proteccion, 272 en total)

  12x TVS gate-source, una por SiC. Sin ella un pico de dv/dt acoplado
      por Cgd puede perforar el oxido de puerta: es el modo de fallo mas
      comun en SiC. Va en el pie del transistor.
  12x snubber RC del nodo de conmutacion (220 pF + 4.7 ohm). El valor sale
      del barrido en LTspice: baja el dv/dt de 147 a 90 V/ns, por debajo
      del CMTI de 100 V/ns del UCC21520, y la sobretension de 823 a 767 V.
   2x TVS en serie sobre el bus DC (5KP440A): recorte en nanosegundos muy
      por delante del chopper, que es un lazo de control.
  12x Schottky de recorte en las entradas de ADC. La R serie del filtro
      anti-alias limita la corriente; sin los diodos, un transitorio de la
      etapa de potencia entra directo al pin del STM32.
   4x TVS de ESD en el conector de campo del ESP32.
   1x polyfuse rearmable + diodo antiinversion + TVS en la entrada de 24 V.

BUGS DESTAPADOS AL CABLEAR LAS PROTECCIONES

  a) Los 4 TVS del conector de campo compartian columna: sus bajadas a
     IOGND se solapaban y cortocircuitaban las cuatro lineas. Cada uno a
     su propia x.
  b) Los diodos de recorte del ADC morian en MITAD del cable de senal, asi
     que KiCad no los conectaba (solo une extremo con extremo, el mismo
     fallo que ya aparecio en los rieles del bus). El cable se parte ahora
     en el punto de recorte.

ASPECTO

  El .kicad_pcb no tenia seccion (stackup), por eso el render salia verde
  por defecto. Se inyecta desde tools/stackup_tpl.txt: mascara negra,
  serigrafia blanca, acabado ENIG (obligado con el LQFP-100 de paso
  0.5 mm) y los espesores reales de cobre (70 um exteriores, 35 um
  interiores) con prepreg fino de 0.2 mm entre F.Cu e In1.Cu para que el
  bus laminado tenga poca inductancia. Los colores son parametros al
  principio de tools/gen_pcb.py.

Co-Authored-By: Claude Opus 5 <noreply@anthropic.com>
Parts:
- added CSNA: 220p 1kV, C_Rect_L24.0mm_W10.3mm_P22.50mm_MKT, F.Cu at (135.2, 88.0)
- added CSNB: 220p 1kV, C_Rect_L24.0mm_W10.3mm_P22.50mm_MKT, F.Cu at (102.7, 107.7)
- added CSNC: 220p 1kV, C_Rect_L24.0mm_W10.3mm_P22.50mm_MKT, F.Cu at (135.2, 107.7)
- added CSNU: 220p 1kV, C_Rect_L24.0mm_W10.3mm_P22.50mm_MKT, F.Cu at (248.7, 88.0)
- added CSNV: 220p 1kV, C_Rect_L24.0mm_W10.3mm_P22.50mm_MKT, F.Cu at (281.2, 88.0)
- added CSNW: 220p 1kV, C_Rect_L24.0mm_W10.3mm_P22.50mm_MKT, F.Cu at (313.6, 88.0)
- added DREV: SS34, D_SMA, F.Cu at (75.7, 162.6)
- added PF1: 2A rearmable, Fuseholder_Blade_ATO_Littelfuse_Pudenz_2_Pin, F.Cu at (42.8, 164.1)
- added RB1H: BAT54, D_SOD-123, F.Cu at (160.0, 178.6)
- added RB1L: BAT54, D_SOD-123, F.Cu at (90.4, 195.1)
- added RB2H: BAT54, D_SOD-123, F.Cu at (99.2, 195.1)
- added RB2L: BAT54, D_SOD-123, F.Cu at (108.0, 195.1)
- added RB3H: BAT54, D_SOD-123, F.Cu at (116.8, 195.1)
- added RB3L: BAT54, D_SOD-123, F.Cu at (125.6, 195.1)
- added RB4H: BAT54, D_SOD-123, F.Cu at (134.4, 195.1)
- added RB4L: BAT54, D_SOD-123, F.Cu at (143.2, 195.1)
- added RB5H: BAT54, D_SOD-123, F.Cu at (152.0, 195.1)
- added RB5L: BAT54, D_SOD-123, F.Cu at (160.8, 195.1)
- added RB6H: BAT54, D_SOD-123, F.Cu at (90.4, 203.2)
- added RB6L: BAT54, D_SOD-123, F.Cu at (99.2, 203.2)
- added RSNA: 4R7 2W, R_2512_6332Metric, F.Cu at (93.9, 123.7)
- added RSNB: 4R7 2W, R_2512_6332Metric, F.Cu at (108.6, 123.7)
- added RSNC: 4R7 2W, R_2512_6332Metric, F.Cu at (123.3, 123.7)
- added RSNU: 4R7 2W, R_2512_6332Metric, F.Cu at (278.5, 104.1)
- added RSNV: 4R7 2W, R_2512_6332Metric, F.Cu at (293.2, 104.1)
- added RSNW: 4R7 2W, R_2512_6332Metric, F.Cu at (307.9, 104.1)
- added TVF1: PESD5V0, D_SOD-123, F.Cu at (320.7, 207.3)
- added TVF2: PESD5V0, D_SOD-123, F.Cu at (329.5, 207.3)
- added TVF3: PESD5V0, D_SOD-123, F.Cu at (276.4, 223.8)
- added TVF4: PESD5V0, D_SOD-123, F.Cu at (285.2, 223.8)
- added TVGH1: +20/-6V, D_SOD-123, F.Cu at (136.6, 123.0)
- added TVGH2: +20/-6V, D_SOD-123, F.Cu at (92.4, 135.5)
- added TVGH3: +20/-6V, D_SOD-123, F.Cu at (104.3, 135.5)
- added TVGH4: +20/-6V, D_SOD-123, F.Cu at (321.2, 103.4)
- added TVGH5: +20/-6V, D_SOD-123, F.Cu at (238.4, 115.8)
- added TVGH6: +20/-6V, D_SOD-123, F.Cu at (250.3, 115.8)
- added TVGL1: +20/-6V, D_SOD-123, F.Cu at (116.1, 135.5)
- added TVGL2: +20/-6V, D_SOD-123, F.Cu at (127.9, 135.5)
- added TVGL3: +20/-6V, D_SOD-123, F.Cu at (139.7, 135.5)
- added TVGL4: +20/-6V, D_SOD-123, F.Cu at (262.1, 115.8)
- added TVGL5: +20/-6V, D_SOD-123, F.Cu at (273.9, 115.8)
- added TVGL6: +20/-6V, D_SOD-123, F.Cu at (285.7, 115.8)
- added TVS1: 5KP440A, D_SMA, F.Cu at (155.5, 32.8)
- added TVS2: 5KP440A, D_SMA, F.Cu at (169.6, 32.8)
- added TVS3: SMBJ33A, D_SMA, F.Cu at (11.5, 179.1)
- moved RB2C 61.6 mm to (106.5, 210.7)
- moved RB1D 61.6 mm to (90.1, 210.7)
- moved RB2B 61.6 mm to (98.3, 210.7)
- moved RB5D 59.4 mm to (106.5, 217.7)
- moved RB5B 59.4 mm to (90.1, 217.7)
- moved RB5C 59.4 mm to (98.3, 217.7)
- moved RLED 59.3 mm to (165.9, 44.3)
- moved RDV6 59.3 mm to (154.3, 44.3)
- moved RB6A 58.9 mm to (98.1, 224.7)
- moved RB5A 58.9 mm to (90.0, 224.7)
- moved RREF 58.9 mm to (106.1, 224.7)
- moved RB1 57.5 mm to (107.9, 203.1)
- moved U42 45.7 mm to (72.1, 179.0)
- moved J50 45.7 mm to (79.9, 182.9)
- moved U41 45.7 mm to (63.9, 179.0)
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Connections:
- F10 pad 2: /09_PSU_Aux_Bias/+24V_F -> Net-(F10-Pad2)
- Q12 pad 3: K_L6 -> DC_N
- Q6 pad 3: K_L3 -> DC_N
- U13 pad 9: K_L3 -> DC_N
- U16 pad 9: K_L6 -> DC_N
