File: kicad/sch/afe_bridge.kicad_sch (KiCad schematic)
At the start: 9 parts, among them Q1 C3M0075120K, Q2 C3M0075120K, Q3 C3M0075120K, Q4 C3M0075120K, Q5 C3M0075120K, Q6 C3M0075120K

Commit message: Corrige tres bugs de conectividad del bus DC y anade guia de simulacion
Al intentar rutear los lazos de conmutacion aparecieron tres errores graves
del esquematico que ninguna revision visual habia detectado:

1. Los rieles del bus DC solo conectaban la ULTIMA rama de cada puente.
   DC_P tenia 4 pads en vez de 22; Q1, Q3, Q7 y Q9 quedaban unconnected.
   Causa: el riel era un unico cable largo y los stubs de cada rama morian
   en mitad de el. KiCad solo une cables extremo con extremo: un cable que
   termina en medio de otro NO conecta, ni con junction. Solo funcionaba la
   ultima rama porque coincidia con el extremo del riel.
   Corregido con un helper rail() que construye el riel PARTIDO en cada
   punto de contacto.

2. El puente AFE no estaba conectado al filtro LCL: el nodo de conmutacion
   se llamaba SW_A y la salida del LCL AFE_A. Mismo nodo fisico, dos
   nombres. Unificado a AFE_A/B/C.

3. La resistencia de precarga quedaba puenteada porque el helper de riel
   se tragaba tambien el nodo DC_RAW. Corregido acotando con xmin.

Resultado: DC_P de 4 a 22 pads, DC_N de 4 a 18.

Tambien: se probo extender el bus laminado sobre toda la fila de potencia y
EMPEORA (293 clearance, 34 cortos): con 3 mm exigidos a HV_DC y los pines
del TO-247-4 a 2.54 mm el plano no cabe entre drenador y puerta. Revertido y
documentado.

Nuevo: docs/COMO_SIMULAR.md con las cuatro simulaciones del proyecto.

Co-Authored-By: Claude Opus 5 <noreply@anthropic.com>
Connections:
- net SW_A renamed AFE_A
- net SW_B renamed AFE_B
- net SW_C renamed AFE_C
Other:
- note added: "SHEET 02 - PUENTE AFE Ramas A/B/C. El nodo de conmutacion ES la salida del LCL (AFE_x). Gates G_H1..3 / G_L1..3 y Kelvin K_H1..3 / K_L1..3 al sheet 05."
- note removed: "SHEET 02 - PUENTE AFE Ramas A/B/C. Nodos SW_A/B/C van al filtro LCL (sheet 01, red AFE_x). Gates G_H1..3 / G_L1..3 y Kelvin K_H1..3 / K_L1..3 al sheet 05."

Commit message: Anade protecciones electricas y stackup con color
PROTECCIONES (de 15 a 56 componentes de proteccion, 272 en total)

  12x TVS gate-source, una por SiC. Sin ella un pico de dv/dt acoplado
      por Cgd puede perforar el oxido de puerta: es el modo de fallo mas
      comun en SiC. Va en el pie del transistor.
  12x snubber RC del nodo de conmutacion (220 pF + 4.7 ohm). El valor sale
      del barrido en LTspice: baja el dv/dt de 147 a 90 V/ns, por debajo
      del CMTI de 100 V/ns del UCC21520, y la sobretension de 823 a 767 V.
   2x TVS en serie sobre el bus DC (5KP440A): recorte en nanosegundos muy
      por delante del chopper, que es un lazo de control.
  12x Schottky de recorte en las entradas de ADC. La R serie del filtro
      anti-alias limita la corriente; sin los diodos, un transitorio de la
      etapa de potencia entra directo al pin del STM32.
   4x TVS de ESD en el conector de campo del ESP32.
   1x polyfuse rearmable + diodo antiinversion + TVS en la entrada de 24 V.

BUGS DESTAPADOS AL CABLEAR LAS PROTECCIONES

  a) Los 4 TVS del conector de campo compartian columna: sus bajadas a
     IOGND se solapaban y cortocircuitaban las cuatro lineas. Cada uno a
     su propia x.
  b) Los diodos de recorte del ADC morian en MITAD del cable de senal, asi
     que KiCad no los conectaba (solo une extremo con extremo, el mismo
     fallo que ya aparecio en los rieles del bus). El cable se parte ahora
     en el punto de recorte.

ASPECTO

  El .kicad_pcb no tenia seccion (stackup), por eso el render salia verde
  por defecto. Se inyecta desde tools/stackup_tpl.txt: mascara negra,
  serigrafia blanca, acabado ENIG (obligado con el LQFP-100 de paso
  0.5 mm) y los espesores reales de cobre (70 um exteriores, 35 um
  interiores) con prepreg fino de 0.2 mm entre F.Cu e In1.Cu para que el
  bus laminado tenga poca inductancia. Los colores son parametros al
  principio de tools/gen_pcb.py.

Co-Authored-By: Claude Opus 5 <noreply@anthropic.com>
Parts:
- added CSNA, CSNB, CSNC: 220p 1kV, Capacitor_THT:C_Rect_L24.0mm_W10.3mm_P22.50mm_MKT, symbol Device:C
- added RSNA, RSNB, RSNC: 4R7 2W, Resistor_SMD:R_2512_6332Metric, symbol Device:R
- added TVGH1, TVGH2, TVGH3, TVGL1, TVGL2, TVGL3: +20/-6V, Diode_SMD:D_SOD-123, symbol Device:D_TVS
Connections:
- net K_L2 is gone; now on net DC_N: Q4.3 (DS)
- net K_L3 is gone; now on net DC_N: Q6.3 (DS)
- net AFE_A: now also CSNA.1
- net AFE_B: now also CSNB.1
- net AFE_C: now also CSNC.1
- net DC_N: now also RSNA.2, RSNB.2, RSNC.2, TVGL2.2 (A2), TVGL3.2 (A2)
- net G_H1: now also TVGH1.1 (A1)
- net G_H2: now also TVGH2.1 (A1)
- net G_H3: now also TVGH3.1 (A1)
- net G_L1: now also TVGL1.1 (A1)
- net G_L2: now also TVGL2.1 (A1)
- net G_L3: now also TVGL3.1 (A1)
- net K_H1: now also TVGH1.2 (A2)
- net K_H2: now also TVGH2.2 (A2)
- net K_H3: now also TVGH3.2 (A2)
- net K_L1: now also TVGL1.2 (A2)
- new net: CSNA.2, RSNA.1
- new net: CSNB.2, RSNB.1
- new net: CSNC.2, RSNC.1
