File: kicad/sch/psu_aux.kicad_sch (KiCad schematic)
At the start: 15 parts, among them J40 24 Vdc IN, J50 DCDC ISO 15V rama 1, J51 DCDC ISO 15V rama 2, J52 DCDC ISO 15V rama 3, J53 DCDC ISO 15V rama 4, J54 DCDC ISO 15V rama 5, J55 DCDC ISO 15V rama 6, U40 LMR33630 24->15V, U41 LMR33630 15->5V, U42 TLV75833 5->3V3

Commit message: Anade protecciones electricas y stackup con color
PROTECCIONES (de 15 a 56 componentes de proteccion, 272 en total)

  12x TVS gate-source, una por SiC. Sin ella un pico de dv/dt acoplado
      por Cgd puede perforar el oxido de puerta: es el modo de fallo mas
      comun en SiC. Va en el pie del transistor.
  12x snubber RC del nodo de conmutacion (220 pF + 4.7 ohm). El valor sale
      del barrido en LTspice: baja el dv/dt de 147 a 90 V/ns, por debajo
      del CMTI de 100 V/ns del UCC21520, y la sobretension de 823 a 767 V.
   2x TVS en serie sobre el bus DC (5KP440A): recorte en nanosegundos muy
      por delante del chopper, que es un lazo de control.
  12x Schottky de recorte en las entradas de ADC. La R serie del filtro
      anti-alias limita la corriente; sin los diodos, un transitorio de la
      etapa de potencia entra directo al pin del STM32.
   4x TVS de ESD en el conector de campo del ESP32.
   1x polyfuse rearmable + diodo antiinversion + TVS en la entrada de 24 V.

BUGS DESTAPADOS AL CABLEAR LAS PROTECCIONES

  a) Los 4 TVS del conector de campo compartian columna: sus bajadas a
     IOGND se solapaban y cortocircuitaban las cuatro lineas. Cada uno a
     su propia x.
  b) Los diodos de recorte del ADC morian en MITAD del cable de senal, asi
     que KiCad no los conectaba (solo une extremo con extremo, el mismo
     fallo que ya aparecio en los rieles del bus). El cable se parte ahora
     en el punto de recorte.

ASPECTO

  El .kicad_pcb no tenia seccion (stackup), por eso el render salia verde
  por defecto. Se inyecta desde tools/stackup_tpl.txt: mascara negra,
  serigrafia blanca, acabado ENIG (obligado con el LQFP-100 de paso
  0.5 mm) y los espesores reales de cobre (70 um exteriores, 35 um
  interiores) con prepreg fino de 0.2 mm entre F.Cu e In1.Cu para que el
  bus laminado tenga poca inductancia. Los colores son parametros al
  principio de tools/gen_pcb.py.

Co-Authored-By: Claude Opus 5 <noreply@anthropic.com>
Parts:
- added DREV: SS34, Diode_SMD:D_SMA, symbol Device:D_Schottky
- added PF1: 2A rearmable, Fuse:Fuseholder_Blade_ATO_Littelfuse_Pudenz_2_Pin, symbol Device:Polyfuse
- added TVS3: SMBJ33A, Diode_SMD:D_SMA, symbol Device:D_TVS
Connections:
- net +15V: now also DREV.2 (A), TVS3.1 (A1)
- net GND: now also TVS3.2 (A2)
- net +24V_F: no longer names the net of F10.2
- net +24V_F: now also PF1.1
- new net: DREV.1 (K), PF1.2
Other:
- note added: "PF1 rearmable + DREV antiinversion + TVS3 de transitorios"
