File: kicad/sch/sense_iv.kicad_sch (KiCad schematic)
At the start: 41 parts, among them J10 HALL AIN_IAFE_A, J11 HALL AIN_IAFE_B, J12 HALL AIN_IAFE_C, J13 HALL AIN_IMOT_U, J14 HALL AIN_IMOT_V, J15 HALL AIN_IMOT_W, U20 LM358

Commit message: Anade protecciones electricas y stackup con color
PROTECCIONES (de 15 a 56 componentes de proteccion, 272 en total)

  12x TVS gate-source, una por SiC. Sin ella un pico de dv/dt acoplado
      por Cgd puede perforar el oxido de puerta: es el modo de fallo mas
      comun en SiC. Va en el pie del transistor.
  12x snubber RC del nodo de conmutacion (220 pF + 4.7 ohm). El valor sale
      del barrido en LTspice: baja el dv/dt de 147 a 90 V/ns, por debajo
      del CMTI de 100 V/ns del UCC21520, y la sobretension de 823 a 767 V.
   2x TVS en serie sobre el bus DC (5KP440A): recorte en nanosegundos muy
      por delante del chopper, que es un lazo de control.
  12x Schottky de recorte en las entradas de ADC. La R serie del filtro
      anti-alias limita la corriente; sin los diodos, un transitorio de la
      etapa de potencia entra directo al pin del STM32.
   4x TVS de ESD en el conector de campo del ESP32.
   1x polyfuse rearmable + diodo antiinversion + TVS en la entrada de 24 V.

BUGS DESTAPADOS AL CABLEAR LAS PROTECCIONES

  a) Los 4 TVS del conector de campo compartian columna: sus bajadas a
     IOGND se solapaban y cortocircuitaban las cuatro lineas. Cada uno a
     su propia x.
  b) Los diodos de recorte del ADC morian en MITAD del cable de senal, asi
     que KiCad no los conectaba (solo une extremo con extremo, el mismo
     fallo que ya aparecio en los rieles del bus). El cable se parte ahora
     en el punto de recorte.

ASPECTO

  El .kicad_pcb no tenia seccion (stackup), por eso el render salia verde
  por defecto. Se inyecta desde tools/stackup_tpl.txt: mascara negra,
  serigrafia blanca, acabado ENIG (obligado con el LQFP-100 de paso
  0.5 mm) y los espesores reales de cobre (70 um exteriores, 35 um
  interiores) con prepreg fino de 0.2 mm entre F.Cu e In1.Cu para que el
  bus laminado tenga poca inductancia. Los colores son parametros al
  principio de tools/gen_pcb.py.

Co-Authored-By: Claude Opus 5 <noreply@anthropic.com>
Parts:
- added RB1H, RB1L, RB2H, RB2L, RB3H, RB3L, RB4H, RB4L, RB5H, RB5L, RB6H, RB6L: BAT54, Diode_SMD:D_SOD-123, symbol Device:D_Schottky
Connections:
- net +3V3: now also RB1H.2 (A), RB2H.2 (A), RB3H.2 (A), RB4H.2 (A), RB5H.2 (A), RB6H.2 (A)
- net AIN_IAFE_A: now also RB1H.1 (K), RB1L.2 (A)
- net AIN_IAFE_B: now also RB2H.1 (K), RB2L.2 (A)
- net AIN_IAFE_C: now also RB3H.1 (K), RB3L.2 (A)
- net AIN_IMOT_U: now also RB4H.1 (K), RB4L.2 (A)
- net AIN_IMOT_V: now also RB5H.1 (K), RB5L.2 (A)
- net AIN_IMOT_W: now also RB6H.1 (K), RB6L.2 (A)
- net GND: now also RB1L.1 (K), RB2L.1 (K), RB3L.1 (K), RB4L.1 (K), RB5L.1 (K), RB6L.1 (K)
